File: Maerklin System Control.kicad_pcb (KiCad board)
At the start: 2 copper layers, 83.8 x 73 mm, 16 parts, among them J1 Female Header, J2 Input, J3 Output, J4 Female Header Left, J5 Female Header Right, Q1 IRF3205, SW1 UP, SW2 RIGHT, SW3 DOWN, SW4 LEFT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

Commit message: latest design
Routing:
- net +5V: track 124.2 -> 87.3 mm, vias 0 -> 1
- net SDA: track 50.1 -> 48.6 mm
- net UP: track 41.2 -> 40.2 mm
- net DIN: track 60.5 -> 61.2 mm
- net MOSFET: track 38.5 -> 37.8 mm

Commit message: latest v1.1 iteration
Parts:
- removed J5: Female Header Right, Connector_PinSocket_2.54mm:PinSocket_2x08_P2.54mm_Vertical
- J4: value Female Header Left -> Conn_S3 Mini; footprint Connector_PinSocket_2.54mm:PinSocket_2x08_P2.54mm_Vertical -> wemos:PinSocket_S3 Mini
- SW1, SW2, SW3, SW4, SW5, SW6: footprint Button_Switch_THT:SW_PUSH_6mm_H4.3mm -> easyeda2kicad:KEY-TH_4P-L6.0-W6.0-P3.90-LS7.8
- moved J4 18.3 mm to (120.5, 44.1)
- moved J3 7.79 mm to (132.1, 88.6)
- moved H1 7.79 mm to (66.6, 27.8)
- moved H3 7.79 mm to (66.6, 90.7)
- moved J1 7.79 mm to (85.9, 38.2)
- moved J2 7.79 mm to (101.4, 88.7)
- moved Q1 7.79 mm to (114.0, 88.4)
- moved SW1 7.79 mm to (82.7, 56.1)
- moved SW2 7.79 mm to (92.5, 65.5)
- moved SW3 7.79 mm to (82.7, 75.4)
- moved SW4 7.79 mm to (72.9, 65.5)
- moved SW5 7.79 mm to (108.0, 75.1)
- moved SW6 7.79 mm to (123.5, 65.5)
- moved H2 7.79 mm to (140.8, 27.9)
- moved H4 7.79 mm to (140.8, 90.7)
Connections:
- net DIN renamed DOUT
- J3 pad 3: GND -> GND1
- J4 pad 10: unconnected-(J4-GPIO7-Pad10) -> LEFT
- J4 pad 11: unconnected-(J4-GPIO11-Pad11) -> RIGHT
- J4 pad 12: unconnected-(J4-GPIO8-Pad12) -> DOWN
- J4 pad 2: UP -> unconnected-(J4-IO2-Pad2)
- J4 pad 4: RIGHT -> unconnected-(J4-IO12-Pad4)
- J4 pad 6: DOWN -> unconnected-(J4-IO11-Pad6)
- J4 pad 8: LEFT -> unconnected-(J4-+3V3-Pad8)
- J4 pad 9: unconnected-(J4-GPIO13-Pad9) -> UP
- Q1 pad 2: GND -> GND1
- SW1 pad 2: GND -> UP
- SW2 pad 2: GND -> RIGHT
- SW3 pad 2: GND -> DOWN
- SW4 pad 2: GND -> LEFT
- SW5 pad 2: GND -> SELECT
- SW6 pad 2: GND -> BACK
Routing:
- net +5V: track 87.3 -> 124.2 mm, vias 1 -> 0
- net GND1: track 0.00 -> 12.0 mm
- net LEFT: track 61.3 -> 51.4 mm
- net DOWN: track 64.5 -> 58.5 mm, vias 1 -> 0
- net BACK: track 19.4 -> 13.9 mm
- net RIGHT: track 46.6 -> 41.3 mm
- net UP: track 40.2 -> 35.3 mm, vias 1 -> 0
- net DOUT: track 61.2 -> 56.5 mm
- net SDA: track 48.6 -> 50.7 mm, vias 1 -> 0
- net SCK: track 47.9 -> 46.2 mm, vias 1 -> 0
- net MOSFET: track 37.8 -> 36.8 mm
Other:
- board text added: "DOUT"
- board text removed: "DIN"

Commit message: start with v1.2
Parts:
- removed Q1: IRF3205, Package_TO_SOT_THT:TO-220-3_Vertical
- added kibuzzard-67897FC0: G***, kibuzzard-67897FC0, B.Cu at (120.4, 43.5)
- added kibuzzard-67898040: G***, kibuzzard-67898040, B.Cu at (75.6, 33.7)
- added kibuzzard-67898062: G***, kibuzzard-67898062, B.Cu at (75.6, 36.3)
- added kibuzzard-67898074: G***, kibuzzard-67898074, B.Cu at (75.6, 38.9)
- added kibuzzard-67898084: G***, kibuzzard-67898084, B.Cu at (75.6, 41.5)
- added kibuzzard-678980A4: G***, kibuzzard-678980A4, B.Cu at (101.4, 94.8)
- added kibuzzard-678980E8: G***, kibuzzard-678980E8, B.Cu at (127.0, 94.8)
- added kibuzzard-678980F4: G***, kibuzzard-678980F4, B.Cu at (122.0, 94.8)
- added kibuzzard-67898102: G***, kibuzzard-67898102, B.Cu at (132.0, 94.8)
- added kibuzzard-678981DB: G***, kibuzzard-678981DB, F.Cu at (108.0, 79.9)
- added kibuzzard-678981FB: G***, kibuzzard-678981FB, F.Cu at (123.4, 70.1)
- added kibuzzard-67898208: G***, kibuzzard-67898208, F.Cu at (82.6, 60.5)
- added kibuzzard-67898217: G***, kibuzzard-67898217, F.Cu at (82.6, 80.1)
- added kibuzzard-67898221: G***, kibuzzard-67898221, F.Cu at (72.8, 70.1)
- added kibuzzard-67898229: G***, kibuzzard-67898229, F.Cu at (92.4, 70.1)
- added kibuzzard-678A131B: G***, kibuzzard-678A131B, B.Cu at (98.8, 82.0)
- added kibuzzard-678A1323: G***, kibuzzard-678A1323, B.Cu at (127.0, 82.0)
- added kibuzzard-678A1332: G***, kibuzzard-678A1332, B.Cu at (96.4, 94.8)
- added kibuzzard-67E5658B: G***, kibuzzard-67E5658B, B.Cu at (81.7, 37.7)
- moved J1 7.64 mm to (79.0, 41.5), turned to 0 degrees
- moved J3 0.30 mm to (132.1, 88.9)
- moved J2 0.18 mm to (101.4, 88.9)
Connections:
- J3 pad 3: GND1 -> GND
- J4 pad 18: MOSFET -> unconnected-(J4-IO37-Pad18)
Routing:
- net +5V: track 124.2 -> 209.2 mm
- net MOSFET: track 36.8 -> 0.00 mm
- net GND1: track 12.0 -> 0.00 mm
- net SELECT: track 26.2 -> 32.7 mm
- net LEFT: track 51.4 -> 57.9 mm
- net BACK: track 13.9 -> 20.4 mm
- net RIGHT: track 41.3 -> 47.7 mm
- net UP: track 35.3 -> 41.7 mm
- net DOWN: track 58.5 -> 63.9 mm
- net DOUT: track 56.5 -> 54.7 mm
- net SDA: track 50.7 -> 50.0 mm
Other:
- board text added: "(c) 2025 by mars3142"
- board text removed: "(c) 2024 by mars3142"
- board text removed: "+5V"
- board text removed: "DOUT"
- board text removed: "GND"
- board text removed: "I2C LCD"
- board text removed: "LOLIN S3 Mini"
- board text removed: "SCK"
- board text removed: "SDA"

Commit message: RC of mk2
Signed-off-by: Peter Siegmund <mars3142@users.noreply.github.com>
Parts:
- removed kibuzzard-67E5658B: G***, kibuzzard-67E5658B
- added C1: 100nF, Capacitor_SMD:C_0805_2012Metric, F.Cu at (115.6, 50.8)
- added C2: 100nF, Capacitor_SMD:C_0805_2012Metric, F.Cu at (124.7, 50.9)
- added C3: 100nF, Capacitor_SMD:C_0805_2012Metric, F.Cu at (133.6, 50.9)
- added D1: WS2812B, LED_SMD:LED_WS2812B_PLCC4_5.0x5.0mm_P3.2mm, F.Cu at (115.6, 46.3)
- added D2: WS2812B, LED_SMD:LED_WS2812B_PLCC4_5.0x5.0mm_P3.2mm, F.Cu at (124.6, 46.3)
- added D3: WS2812B, LED_SMD:LED_WS2812B_PLCC4_5.0x5.0mm_P3.2mm, F.Cu at (133.6, 46.3)
- added kibuzzard-6859B258: G***, kibuzzard-6859B258, B.Cu at (77.3, 51.9)
- moved kibuzzard-67897FC0 26.0 mm to (129.6, 67.7), turned to 90 degrees
- moved J4 24.1 mm to (124.6, 67.9), turned to 180 degrees
- moved H1 18.1 mm to (67.6, 45.9)
- moved H2 17.9 mm to (140.6, 45.9)
- moved kibuzzard-67898074 14.9 mm to (71.2, 53.1)
- moved kibuzzard-67898084 14.9 mm to (71.2, 55.7)
- moved kibuzzard-67898040 14.9 mm to (71.2, 47.9)
- moved kibuzzard-67898062 14.9 mm to (71.2, 50.5)
- moved J1 14.9 mm to (74.6, 55.7)
- moved kibuzzard-678981DB 10.7 mm to (111.0, 90.2)
- moved SW5 10.4 mm to (110.6, 85.2)
- moved kibuzzard-678981FB 9.77 mm to (123.4, 79.8)
- moved kibuzzard-67898208 9.77 mm to (82.6, 70.2)
- moved kibuzzard-67898217 9.77 mm to (82.6, 89.8)
- moved kibuzzard-67898221 9.77 mm to (72.8, 79.8)
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- renumbered J3 to J2, J2 to J3
Connections:
- J4 pad 2: unconnected-(J4-IO2-Pad2) -> LED
Routing:
- net +5V: track 209.2 -> 139.6 mm, vias 0 -> 1
- net DOUT: track 54.7 -> 15.0 mm
- net LED: track 0.00 -> 27.4 mm
- net LEFT: track 57.9 -> 78.3 mm, vias 0 -> 1
- net DOWN: track 63.9 -> 81.6 mm
- net UP: track 41.7 -> 58.0 mm
- net Net-(D1-DOUT): track 0.00 -> 15.9 mm, vias 0 -> 2
- net Net-(D2-DOUT): track 0.00 -> 15.3 mm
- net SELECT: track 32.7 -> 25.8 mm
- net BACK: track 20.4 -> 15.9 mm
- net SDA: track 50.0 -> 54.5 mm
- net Net-(D3-VSS): track 0.00 -> 3.52 mm
- net Net-(D1-VSS): track 0.00 -> 3.51 mm
- net Net-(D2-VSS): track 0.00 -> 3.48 mm
- net SCK: track 46.4 -> 49.6 mm
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Other:
- board size 83.8 x 73 mm -> 83 x 55 mm
- board text added: "System Control MK2"
- board text removed: "JLCJLCJLCJLC"
- board text removed: "System Control MK1.1"
