File: Maerklin System Control.kicad_pcb (KiCad board)
At the start: 2 copper layers, 83 x 55 mm, 39 parts, among them J1 Female Header, J2 Output, J3 Input, J4 Conn_S3 Mini, SW1 UP, SW2 RIGHT, SW3 DOWN, SW4 LEFT, SW5 SELECT, SW6 BACK

Commit message: FIX: WLED connection
Signed-off-by: Peter Siegmund <mars3142@users.noreply.github.com>
Parts:
- C1, C2, C3: footprint Capacitor_SMD:C_0805_2012Metric -> Capacitor_SMD:C_0805_2012Metric_Pad1.18x1.45mm_HandSolder
- moved C3 20.3 mm to (114.4, 44.4), turned to 0 degrees
- moved D3 17.9 mm to (115.9, 48.4)
- moved D1 17.4 mm to (132.9, 48.4)
- moved C1 17.0 mm to (131.4, 44.4), turned to 0 degrees
- moved C2 6.75 mm to (122.9, 44.4), turned to 0 degrees
- moved D2 2.06 mm to (124.4, 48.4)
Connections:
- C1 pad 1: Net-(D1-VSS) -> +5V
- C2 pad 1: Net-(D2-VSS) -> +5V
- C3 pad 1: Net-(D3-VSS) -> +5V
- D1 pad 3: Net-(D1-VSS) -> GND
- D2 pad 3: Net-(D2-VSS) -> GND
- D3 pad 3: Net-(D3-VSS) -> GND
Routing:
- net +5V: track 139.6 -> 211.4 mm, vias 1 -> 2
- net LED: track 27.4 -> 16.1 mm
- net Net-(D1-DOUT): track 15.9 -> 4.92 mm, vias 2 -> 0
- net Net-(D2-DOUT): track 15.3 -> 5.02 mm
- net Net-(D3-VSS): track 3.52 -> 0.00 mm
- net Net-(D1-VSS): track 3.51 -> 0.00 mm
- net Net-(D2-VSS): track 3.48 -> 0.00 mm
Other:
- board text added: "System Control MK2.1"
- board text removed: "System Control MK2"
