File: Maerklin System Control.kicad_sch (KiCad schematic)
At the start: 16 parts, among them J1 Female Header, J2 Input, J3 Output, J4 Female Header Left, J5 Female Header Right, Q1 IRF3205, SW1 UP, SW2 RIGHT, SW3 DOWN, SW4 LEFT, SW5 SELECT, SW6 BACK

Commit message: latest design
Other:
- note added: "Hole"
Changed lines of the file:
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@@
+		)
+	)
+	(text "Hole"
+		(exclude_from_sim no)
+		(at 42.672 56.896 0)
+		(effects
+			(font
+				(size 1.27 1.27)
+			)
 		)
 	)
 	(text "Power / Data"
 		(exclude_from_sim no)
-		(at 90.424 20.574 0)
+		(at 89.408 20.066 0)
 		(effects
 			(font
@@
 		(dnp no)
 		(property "Reference" "SW3"
-			(at 60.96 91.44 0)
+			(at 60.706 92.71 0)
 			(effects
 				(font
@@
 		)
 		(property "Value" "DOWN"
-			(at 60.96 93.98 0)
+			(at 60.706 95.25 0)
 			(effects
 				(font
@@
 	)
 	(symbol
+		(lib_name "SW_Push_Dual_x2_2")
 		(lib_id "Switch:SW_Push_Dual_x2")
 		(at 26.67 100.33 0)
@@
 	)
 	(symbol
+		(lib_name "SW_Push_Dual_x2_1")
 		(lib_id "Switch:SW_Push_Dual_x2")
 		(at 44.45 100.33 0)

Commit message: latest v1.1 iteration
Parts:
- removed J4: Female Header Left, Connector_PinSocket_2.54mm:PinSocket_2x08_P2.54mm_Vertical, symbol Connector_Generic:Conn_02x08_Counter_Clockwise
- removed J5: Female Header Right, Connector_PinSocket_2.54mm:PinSocket_2x08_P2.54mm_Vertical, symbol Connector_Generic:Conn_02x08_Counter_Clockwise
- added J4: Conn_S3 Mini, wemos:PinSocket_S3 Mini, symbol wemos:Conn_S3 Mini
- J2: LCSC C5188434 -> (none); LCSC Part (none) -> C5188434
- J3: LCSC C5188435 -> (none); LCSC Part (none) -> C5188435
- SW1, SW2, SW3, SW5, SW6: footprint Button_Switch_THT:SW_PUSH_6mm_H4.3mm -> easyeda2kicad:KEY-TH_4P-L6.0-W6.0-P3.90-LS7.8; symbol Switch:SW_Push_Dual_x2 -> easyeda2kicad:K2-6639DP-B4SW-04; LCSC C83205 -> (none); LCSC Part (none) -> C83205
- SW4: footprint Button_Switch_THT:SW_PUSH_6mm_H4.3mm -> easyeda2kicad:KEY-TH_4P-L6.0-W6.0-P3.90-LS7.8; symbol Switch:SW_Push_Dual_x2 -> easyeda2kicad:K2-6639DP-B4SW-04; LCSC Part (none) -> C83205
Connections:
- net +5V: now also J4.32 (VBUS)
- net BACK: now also SW6.2, J4.30 (IO16)
- net DOWN: now also SW3.2, J4.12 (IO6)
- net GND: now also SW1.3, SW1.4, SW2.3, SW2.4, SW3.3, SW3.4, SW4.3, SW4.4, SW5.3, SW5.4, SW6.3, SW6.4, J4.23 (GND), J4.31 (GND); no longer J3.3 (Pin_3), Q1.2 (D), SW1.2 (D), SW2.2 (D), SW3.2 (D), SW4.2 (D), SW5.2 (D), SW6.2 (D)
- net LEFT: now also SW4.2, J4.10 (IO3)
- net MOSFET: now also J4.18 (IO37)
- net RIGHT: now also SW2.2, J4.11 (IO5)
- net SCK: now also J4.27 (IO36)
- net SDA: now also J4.28 (IO35)
- net SELECT: now also SW5.2, J4.29 (IO18)
- net UP: now also SW1.2, J4.9 (IO1)
- net DIN renamed DOUT
- net DOUT: now also J4.16 (IO14)
- new net GND1: J3.3 (Pin_3), Q1.2 (D)
Other:
- note added: "Holes"
- note removed: "Hole"
- company: Peter Siegmund (mars3142) -> mars3142
- moved on the sheet: J1

Commit message: start with v1.2
Parts:
- removed Q1: IRF3205, Package_TO_SOT_THT:TO-220-3_Vertical, symbol Transistor_FET:IRF3205
Connections:
- net GND1 is gone; now on net GND: J3.3 (Pin_3)
- net MOSFET: no longer names the net of J4.18 (IO37)
- no-connect marks 19 -> 20
Other:
- moved on the sheet: H1, H2, H3, H4, J2, J3, J4

Commit message: RC of mk2
Signed-off-by: Peter Siegmund <mars3142@users.noreply.github.com>
Parts:
- added C1, C2, C3: 100nF, Capacitor_SMD:C_0805_2012Metric, symbol Device:C
- added D1, D2, D3: WS2812B, LED_SMD:LED_WS2812B_PLCC4_5.0x5.0mm_P3.2mm, symbol LED:WS2812B
- renumbered J3 to J2, J2 to J3
Connections:
- net +5V: now also D1.1 (VDD), D2.1 (VDD), D3.1 (VDD)
- net GND: now also C1.2, C2.2, C3.2
- net LED: now reaches J4.2 (IO2)
- net LED: now also D1.4 (DIN)
- new net: C2.1, D2.3 (VSS)
- new net: D1.2 (DOUT), D2.4 (DIN)
- new net: C1.1, D1.3 (VSS)
- new net: C3.1, D3.3 (VSS)
- new net: D2.2 (DOUT), D3.4 (DIN)
- no-connect marks 20 -> 19
Other:
- note added: "I2C OLED Display"
- note added: "Status LEDs"
- note removed: "I2C LCD"
- moved on the sheet: J1, J2, J3, SW1, SW2, SW3, SW4, SW5, SW6
